File: _autosave-EE475_PCB.kicad_sch (KiCad schematic)
At the start: 11 parts, among them J1 Conn_01x15_Female, J2 Conn_01x02_Female, J3 Conn_01x15_Female, J4 Conn_01x02_Female, Q1 S8050, Q2 S8050

Commit message: Motor Controller Hub PCB Design Update. Added new schematic and layout
Parts:
- J2, J4: footprint (none) -> Connector_PinSocket_2.54mm:PinSocket_1x02_P2.54mm_Vertical
Changed lines of the file:
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@@
       (effects (font (size 1.27 1.27)) (justify left))
     )
-    (property "Footprint" "" (id 2) (at 199.39 38.735 0)
+    (property "Footprint" "Connector_PinSocket_2.54mm:PinSocket_1x02_P2.54mm_Vertical" (id 2) (at 199.39 38.735 0)
       (effects (font (size 1.27 1.27)) hide)
     )
@@
       (effects (font (size 1.27 1.27)) (justify left))
     )
-    (property "Footprint" "" (id 2) (at 151.765 38.1 0)
+    (property "Footprint" "Connector_PinSocket_2.54mm:PinSocket_1x02_P2.54mm_Vertical" (id 2) (at 151.765 38.1 0)
       (effects (font (size 1.27 1.27)) hide)
     )
@@
     )
     (path "/b6ce3de8-74e3-4d01-b190-d0274582e099"
-      (reference "J2") (unit 1) (value "Conn_01x02_Female") (footprint "")
+      (reference "J2") (unit 1) (value "Conn_01x02_Female") (footprint "Connector_PinSocket_2.54mm:PinSocket_1x02_P2.54mm_Vertical")
     )
     (path "/d09b42b3-a1d3-4700-b9ed-e9258430cad0"
@@
     )
     (path "/7d8d3fcc-1fb1-4da8-b4f9-db58981f1c77"
-      (reference "J4") (unit 1) (value "Conn_01x02_Female") (footprint "")
+      (reference "J4") (unit 1) (value "Conn_01x02_Female") (footprint "Connector_PinSocket_2.54mm:PinSocket_1x02_P2.54mm_Vertical")
     )
     (path "/41cec304-98be-4691-a921-3c7db05a2fbc"
