File: EE475_PCB.kicad_sch (KiCad schematic)
At the start: 16 parts, among them J1 Conn_01x15_Female, J2 Conn_01x02_Female, J3 Conn_01x15_Female, J4 Conn_01x02_Female, J5 Conn_01x02_Female, J6 Conn_01x02_Female, J7 Conn_01x02_Female, J8 Conn_01x02_Female, Q1 S8050, Q2 S8050

Commit message: Modify LED and resistor footprint
Parts:
- removed D3: LED_BGRK, LED_SMD:LED_RGB_1210, symbol Device:LED_BGRK
- added D3: LED_RGBA, LED_SMD:LED_RGB_1210, symbol Device:LED_RGBA
- R1, R2, R3: footprint Resistor_SMD:R_0402_1005Metric -> Resistor_SMD:R_1206_3216Metric
Connections:
- net at R2.1: now also D3.2 (GK)
- net at R1.1: now also D3.1 (RK)
- net at J1.2 (Pin_2): now also D3.4 (A)
- net at R3.1: now also D3.3 (BK)
- no-connect marks 28 -> 27
Changed lines of the file:
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@@
   (junction (at 73.025 138.43) (diameter 0) (color 0 0 0 0)
-  )
-  (junction (at 194.31 70.485) (diameter 0) (color 0 0 0 0)
   )
   (junction (at 97.79 126.365) (diameter 0) (color 0 0 0 0)
@@
   (no_connect (at 173.355 102.87))
   (no_connect (at 173.355 123.19))
-  (no_connect (at 107.95 95.885))
   (no_connect (at 173.355 128.27))
   (no_connect (at 107.95 100.965))
@@
     (stroke (width 0) (type default) (color 0 0 0 0))
   )
+  (wire (pts (xy 107.95 95.885) (xy 102.87 95.885))
+    (stroke (width 0) (type default) (color 0 0 0 0))
+  )
   (wire (pts (xy 78.74 126.365) (xy 59.055 126.365))
     (stroke (width 0) (type default) (color 0 0 0 0))
@@
     (stroke (width 0) (type default) (color 0 0 0 0))
   )
+  (wire (pts (xy 213.36 83.82) (xy 213.36 96.52))
+    (stroke (width 0) (type default) (color 0 0 0 0))
+  )
   (wire (pts (xy 85.09 140.97) (xy 85.09 126.365))
     (stroke (width 0) (type default) (color 0 0 0 0))
@@
     (stroke (width 0) (type default) (color 0 0 0 0))
   )
-  (wire (pts (xy 213.36 96.52) (xy 213.36 70.485))
-    (stroke (width 0) (type default) (color 0 0 0 0))
-  )
   (wire (pts (xy 78.74 151.13) (xy 78.74 126.365))
     (stroke (width 0) (type default) (color 0 0 0 0))
@@
     (stroke (width 0) (type default) (color 0 0 0 0))
   )
-  (wire (pts (xy 194.31 60.96) (xy 194.31 70.485))
+  (wire (pts (xy 194.31 60.96) (xy 194.31 80.01))
     (stroke (width 0) (type default) (color 0 0 0 0))
   )
@@
     (stroke (width 0) (type default) (color 0 0 0 0))
   )
+  (wire (pts (xy 102.87 83.82) (xy 213.36 83.82))
+    (stroke (width 0) (type default) (color 0 0 0 0))
+  )
+  (wire (pts (xy 102.87 95.885) (xy 102.87 83.82))
+    (stroke (width 0) (type default) (color 0 0 0 0))
+  )
   (wire (pts (xy 89.535 151.13) (xy 78.74 151.13))
     (stroke (width 0) (type default) (color 0 0 0 0))
@@
     (stroke (width 0) (type default) (color 0 0 0 0))
   )
-  (wire (pts (xy 194.31 70.485) (xy 194.31 80.01))
-    (stroke (width 0) (type default) (color 0 0 0 0))
-  )
   (wire (pts (xy 186.69 55.88) (xy 179.07 55.88))
     (stroke (width 0) (type default) (color 0 0 0 0))
@@
   )
   (wire (pts (xy 146.685 40.64) (xy 137.16 40.64))
-    (stroke (width 0) (type default) (color 0 0 0 0))
-  )
-  (wire (pts (xy 213.36 70.485) (xy 194.31 70.485))
     (stroke (width 0) (type default) (color 0 0 0 0))
   )
@@
     (property "Reference" "R2" (id 0) (at 191.135 91.44 90))
     (property "Value" "1k" (id 1) (at 191.135 93.98 90))
-    (property "Footprint" "Resistor_SMD:R_0402_1005Metric" (id 2) (at 191.135 97.155 0)
+    (property "Footprint" "Resistor_SMD:R_1206_3216Metric" (id 2) (at 191.135 97.155 0)
       (effects (font (size 1.27 1.27)) hide)
     )
@@
     (property "Reference" "R1" (id 0) (at 186.055 88.9 90))
     (property "Value" "1k" (id 1) (at 186.055 91.44 90))
-    (property "Footprint" "Resistor_SMD:R_0402_1005Metric" (id 2) (at 186.055 94.615 0)
+    (property "Footprint" "Resistor_SMD:R_1206_3216Metric" (id 2) (at 186.055 94.615 0)
       (effects (font (size 1.27 1.27)) hide)
     )
@@
     (pin "2")
     (pin "3")
+  )
+  (symbol (lib_id "Device:LED_RGBA") (at 208.28 96.52 0) (unit 1)
+    (in_bom yes) (on_board yes) (fields_autoplaced)
+    (property "Reference" "D3" (id 0) (at 208.28 82.55 0))
+    (property "Value" "LED_RGBA" (id 1) (at 208.28 85.09 0))
+    (property "Footprint" "LED_SMD:LED_RGB_1210" (id 2) (at 208.28 97.79 0)
+      (effects (font (size 1.27 1.27)) hide)
+    )
+    (property "Datasheet" "~" (id 3) (at 208.28 97.79 0)
+      (effects (font (size 1.27 1.27)) hide)
+    )
+    (pin "1")
+    (pin "2")
+    (pin "3")
+    (pin "4")
   )
   (symbol (lib_id "Diode:1N4007") (at 120.015 36.195 270) (unit 1)
@@
     (pin "3")
   )
-  (symbol (lib_id "Device:LED_BGRK") (at 208.28 96.52 0) (mirror y) (unit 1)
-    (in_bom yes) (on_board yes) (fields_autoplaced)
-    (property "Reference" "D3" (id 0) (at 208.28 82.55 0))
-    (property "Value" "LED_BGRK" (id 1) (at 208.28 85.09 0))
-    (property "Footprint" "LED_SMD:LED_RGB_1210" (id 2) (at 208.28 97.79 0)
-      (effects (font (size 1.27 1.27)) hide)
-    )
-    (property "Datasheet" "~" (id 3) (at 208.28 97.79 0)
-      (effects (font (size 1.27 1.27)) hide)
-    )
-    (pin "1")
-    (pin "2")
-    (pin "3")
-    (pin "4")
-  )
   (symbol (lib_id "Device:R_Small_US") (at 196.85 100.965 270) (unit 1)
     (in_bom yes) (on_board yes) (fields_autoplaced)
     (property "Reference" "R3" (id 0) (at 196.85 95.25 90))
     (property "Value" "1k" (id 1) (at 196.85 97.79 90))
-    (property "Footprint" "Resistor_SMD:R_0402_1005Metric" (id 2) (at 196.85 100.965 0)
+    (property "Footprint" "Resistor_SMD:R_1206_3216Metric" (id 2) (at 196.85 100.965 0)
       (effects (font (size 1.27 1.27)) hide)
     )
@@
       (reference "D2") (unit 1) (value "1N4007") (footprint "Diode_THT:D_DO-41_SOD81_P10.16mm_Horizontal")
     )
-    (path "/dcd044fc-a554-401a-b772-5418f9b2ea05"
-      (reference "D3") (unit 1) (value "LED_BGRK") (footprint "LED_SMD:LED_RGB_1210")
+    (path "/45ff345d-8bf2-4568-9463-fbbb7817f5b9"
+      (reference "D3") (unit 1) (value "LED_RGBA") (footprint "LED_SMD:LED_RGB_1210")
     )
     (path "/5f1a4039-9dd3-4da9-ba86-1190356554ff"
@@
     )
     (path "/1fa34a24-9490-47ea-9f6f-3b46a7521208"
-      (reference "R1") (unit 1) (value "1k") (footprint "Resistor_SMD:R_0402_1005Metric")
+      (reference "R1") (unit 1) (value "1k") (footprint "Resistor_SMD:R_1206_3216Metric")
     )
     (path "/159d42a8-6e73-481f-bf76-fc0977179af5"
-      (reference "R2") (unit 1) (value "1k") (footprint "Resistor_SMD:R_0402_1005Metric")
+      (reference "R2") (unit 1) (value "1k") (footprint "Resistor_SMD:R_1206_3216Metric")
     )
     (path "/e39de572-5374-4de1-ac89-4ccec206d5ac"
-      (reference "R3") (unit 1) (value "1k") (footprint "Resistor_SMD:R_0402_1005Metric")
-    )
-  )
+      (reference "R3") (unit 1) (value "1k") (footprint "Resistor_SMD:R_1206_3216Metric")
+    )
+  )
